Commit message: Updated xacro and gazebo files

File: catkin_ws/src/my_robot/urdf/my_robot.xacro (robot description, xacro)
@@ -173,3 +173,10 @@
     </visual>
   </link>
+  <joint name="camera_optical_joint" type="fixed">
+    <origin xyz="0 0 0" rpy="-1.5707 0 -1.5707"/>
+    <parent link="camera_link"/>
+    <child link="camera_link_optical"/>
+  </joint>
+  <link name="camera_link_optical">
+  </link>
 </robot>

Commit message: Update my_robot xacro and urdf files to improve robot camera

File: catkin_ws/src/my_robot/urdf/my_robot.xacro (robot description, xacro)
@@ -120,5 +120,5 @@
   <joint type="fixed" name="camera_joint">
     <origin xyz="0.2 0 0" rpy="0 0 0"/>
-    <child link="camera"/>
+    <child link="camera_link"/>
     <parent link="chassis"/>
     <axis xyz="0 1 0" rpy="0 0 0"/>
@@ -126,5 +126,5 @@
     <dynamics damping="1.0" friction="1.0"/>
   </joint>
-  <link name="camera">
+  <link name="camera_link"> <!--Updated the link name from "camera" to "camera_link"-->
     <inertial>
       <mass value="0.1"/>
